Commit message: Added EKF

File: mobile_robot_unal_description/urdf/mobile_base.gazebo.xacro (robot description, xacro)
@@ -21,3 +21,31 @@
         <fdir1>0 0 1</fdir1>
     </gazebo>
+    <gazebo>
+        <plugin name="imu_plugin" filename="libgazebo_ros_imu.so">
+            <alwaysOn>true</alwaysOn>
+            <bodyName>$(arg robot_name)/imu_link</bodyName>
+            <frameName>$(arg robot_name)/imu_link</frameName>
+            <topicName>imu_data</topicName>
+            <serviceName>imu_service</serviceName>
+            <gaussianNoise>0.05</gaussianNoise>
+            <updateRate>500</updateRate>
+            <imu>
+                <noise>
+                <type>gaussian</type>
+                <rate>
+                    <mean>0.0</mean>
+                    <stddev>2e-4</stddev>
+                    <bias_mean>0.0000075</bias_mean>
+                    <bias_stddev>0.0000008</bias_stddev>
+                </rate>
+                <accel>
+                    <mean>0.0</mean>
+                    <stddev>1.7e-2</stddev>
+                    <bias_mean>0.1</bias_mean>
+                    <bias_stddev>0.001</bias_stddev>
+                </accel>
+                </noise>
+            </imu>
+        </plugin>
+    </gazebo>
 </robot>

File: mobile_robot_unal_description/urdf/mobile_base.urdf.xacro (robot description, xacro)
@@ -146,4 +146,12 @@
         </inertial>
     </link>
+    <!-- IMU Joint (attaching mobile_base_link and imu_link)-->
+    <joint name="imu_joint" type="fixed">
+        <parent link="$(arg robot_name)/mobile_base_link"/>
+        <child link="$(arg robot_name)/imu_link"/>
+        <origin xyz="0.0 -0.06 0.10" rpy="0 0 0"/>
+    </joint>
+    <!-- IMU Link description -->
+    <link name="$(arg robot_name)/imu_link"/>
     <!-- #################################################################################### -->
     <!-- Platform to attach manipulator-->
