Commit message: Change manipulator description to conform to DH parameters

File: manipulator_unal_description/urdf/manipulator_backup.urdf.xacro (robot description, xacro)
@@ -90,7 +90,7 @@
     <!-- Shoulder Joint (attaching shoulder_link and upper_arm_link)-->
     <joint name="shoulder_joint" type="revolute">
-        <axis xyz="0 0 1"/>
+        <axis xyz="0 1 0"/>
         <limit effort="100" lower="${radians(-106)}" upper="${radians(101)}" velocity="${pi}"/>
-        <origin rpy="${-pi/2} 0 0" xyz="0 0 0.04805"/>
+        <origin rpy="0 0 0" xyz="0 0 0.04805"/>
         <parent link="$(arg robot_name)/shoulder_link"/>
         <child link="$(arg robot_name)/upper_arm_link"/>
@@ -99,5 +99,5 @@
     <link name="$(arg robot_name)/upper_arm_link">
         <visual>
-            <origin rpy="${pi/2} ${-pi/2} 0" xyz="0 0 0"/>
+            <origin rpy="0 0 ${pi/2}" xyz="0 0 0"/>
             <geometry>
                 <mesh filename="package://manipulator_unal_description/meshes/VXSA-300-M-3-UA.stl" scale="0.001 0.001 0.001"/>
@@ -106,5 +106,5 @@
         </visual>
         <collision>
-            <origin rpy="${pi/2} ${-pi/2} 0" xyz="0 0 0"/>
+            <origin rpy="0 0 ${pi/2}" xyz="0 0 0"/>
             <geometry>
                 <mesh filename="package://manipulator_unal_description/meshes/VXSA-300-M-3-UA.stl" scale="0.001 0.001 0.001"/>
@@ -112,5 +112,5 @@
         </collision>
         <inertial>
-            <origin rpy="${pi/2} ${-pi/2} 0" xyz="0.0206949000 -0.2264590000 0.0000000004"/>
+            <origin rpy="0 0 ${pi/2}" xyz="0.0206949000 0.0000000004 0.2264590000"/>
             <mass value="0.792592" />
             <inertia    ixx="0.0089250000"
@@ -124,7 +124,7 @@
     <!-- Elbow Joint (attaching upper_arm_link and upper_forearm_link)-->
     <joint name="elbow_joint" type="revolute">
-        <axis xyz="0 0 1"/>
+        <axis xyz="0 1 0"/>
         <limit effort="100" lower="${radians(-92)}" upper="${radians(101)}" velocity="${pi}"/>
-        <origin rpy="${pi} 0 0" xyz="0.05955 -0.3 0.0"/>
+        <origin rpy="${pi} 0 0" xyz="0.05955 0 0.3"/>
         <parent link="$(arg robot_name)/upper_arm_link"/>
         <child link="$(arg robot_name)/upper_forearm_link"/>
@@ -133,5 +133,5 @@
     <link name="$(arg robot_name)/upper_forearm_link">
         <visual>
-            <origin rpy="${pi/2} 0 0" xyz="0 0 0"/>
+            <origin rpy="0 0 0" xyz="0 0 0"/>
             <geometry>
                 <mesh filename="package://manipulator_unal_description/meshes/VXSA-300-M-4-UF.stl" scale="0.001 0.001 0.001"/>
@@ -140,5 +140,5 @@
         </visual>
         <collision>
-            <origin rpy="${pi/2} 0 0" xyz="0 0 0"/>
+            <origin rpy="0 0 0" xyz="0 0 0"/>
             <geometry>
                 <mesh filename="package://manipulator_unal_description/meshes/VXSA-300-M-4-UF.stl" scale="0.001 0.001 0.001"/>
@@ -146,5 +146,5 @@
         </collision>
         <inertial>
-            <origin rpy="${pi/2} 0 0" xyz="0.105723 0 0"/>
+            <origin rpy="0 0 0" xyz="0.105723 0 0"/>
             <mass value="0.322228" />
             <inertia    ixx="0.0001524000"
@@ -158,7 +158,7 @@
     <!-- Upper Forearm Joint (attaching upper_forearm_link and lowe_forearm_link)-->
     <joint name="upper_forearm_joint" type="revolute">
-        <axis xyz="0 0 1"/>
+        <axis xyz="1 0 0"/>
         <limit effort="100" lower="${radians(-180)}" upper="${radians(180)}" velocity="${pi}"/>
-        <origin rpy="${pi/2} 0 ${pi/2}" xyz="0.2 0 0"/>
+        <origin rpy="0 0 0" xyz="0.2 0 0"/>
         <parent link="$(arg robot_name)/upper_forearm_link"/>
         <child link="$(arg robot_name)/lower_forearm_link"/>
@@ -167,5 +167,5 @@
     <link name="$(arg robot_name)/lower_forearm_link">
         <visual>
-            <origin rpy="0 ${-pi/2} 0" xyz="0 0 0"/>
+            <origin rpy="0 0 0" xyz="0 0 0"/>
             <geometry>
                 <mesh filename="package://manipulator_unal_description/meshes/VXSA-300-M-5-LF.stl" scale="0.001 0.001 0.001"/>
@@ -174,5 +174,5 @@
         </visual>
         <collision>
-            <origin rpy="0 ${-pi/2} 0" xyz="0 0 0"/>
+            <origin rpy="0 0 0" xyz="0 0 0"/>
             <geometry>
                 <mesh filename="package://manipulator_unal_description/meshes/VXSA-300-M-5-LF.stl" scale="0.001 0.001 0.001"/>
@@ -180,5 +180,5 @@
         </collision>
         <inertial>
-            <origin rpy="0 ${-pi/2} 0" xyz="0 -0.0068046200 0.0513477000"/>
+            <origin rpy="0 0 0" xyz="0.0513477000 -0.0068046200 0"/>
             <mass value="0.414823" />
             <inertia    ixx="0.0001753000"
@@ -192,7 +192,7 @@
     <!-- Lower Forearm Joint (attaching lower_forearm_link and wrist_link)-->
     <joint name="lower_forearm_joint" type="revolute">
-        <axis xyz="0 0 1"/>
+        <axis xyz="0 1 0"/>
         <limit effort="100" lower="${radians(-130)}" upper="${radians(107)}" velocity="${pi}"/>
-        <origin rpy="${-pi/2} ${-pi/2} 0" xyz="0 0 0.1"/>
+        <origin rpy="0 0 0" xyz="0.1 0 0"/>
         <parent link="$(arg robot_name)/lower_forearm_link"/>
         <child link="$(arg robot_name)/wrist_link"/>
@@ -201,5 +201,5 @@
     <link name="$(arg robot_name)/wrist_link">
         <visual>
-            <origin rpy="0 ${pi/2} ${pi/2}" xyz="0 0 0"/>
+            <origin rpy="0 ${pi} ${pi/2}" xyz="0 0 0"/>
             <geometry>
                 <mesh filename="package://manipulator_unal_description/meshes/VXSA-300-M-6-Wrist.stl" scale="0.001 0.001 0.001"/>
@@ -214,5 +214,5 @@
         </collision>
         <inertial>
-            <origin rpy="0 ${pi} ${pi/2}" xyz="0.0467430000 0.0105650000 0.0000076652"/>
+            <origin rpy="0 ${pi} ${pi/2}" xyz="0.0467430000 0.0000076652 -0.0105650000"/>
             <mass value="0.115395" />
             <inertia    ixx="0.0000463100"
@@ -226,7 +226,7 @@
     <!-- Wrist Joint (attaching wrist_link and gripper)-->
     <joint name="wrist_joint" type="revolute">
-        <axis xyz="0 0 1"/>
+        <axis xyz="1 0 0"/>
         <limit effort="100" lower="${-pi}" upper="${pi}" velocity="${pi}"/>
-        <origin rpy="${-pi/2} 0 ${-pi/2}" xyz="0.069744 0 0"/>
+        <origin rpy="${-pi} 0 0" xyz="0.069744 0 0"/>
         <parent link="$(arg robot_name)/wrist_link"/>
         <child link="$(arg robot_name)/base_gripper_link"/>
@@ -235,5 +235,5 @@
     <link name="$(arg robot_name)/base_gripper_link">
         <visual>
-            <origin rpy="${pi/2} ${pi} ${-pi/2}" xyz="0 0 -0.02"/>
+            <origin rpy="0 0 ${pi/2}" xyz="-0.02 0 0"/>
             <geometry>
                 <mesh filename="package://manipulator_unal_description/meshes/VXSA-300-M-7-Gripper.stl" scale="0.001 0.001 0.001"/>
@@ -242,5 +242,5 @@
         </visual>
         <collision>
-            <origin rpy="${pi/2} ${pi} ${-pi/2}" xyz="-0.02 0 0"/>
+            <origin rpy="0 0 ${pi/2}" xyz="-0.02 0 0"/>
             <geometry>
                 <mesh filename="package://manipulator_unal_description/meshes/VXSA-300-M-7-Gripper.stl" scale="0.001 0.001 0.001"/>
@@ -248,5 +248,5 @@
         </collision>
         <inertial>
-            <origin rpy="${pi/2} ${pi} ${-pi/2}" xyz="-0.0115230000  0.0000000000 0.0230010000"/>
+            <origin rpy="0 0 ${pi/2}" xyz="0.0230010000 0.0000000000 0.0115230000"/>
             <mass value="0.097666" />
             <inertia    ixx="0.0000326800"
@@ -260,5 +260,6 @@
     <!-- Fixed joint to End Effector-->
     <joint name="tcp_joint" type="fixed">
-        <origin rpy="0 ${-pi/2} 0" xyz="0.0 0 0.042825"/>
+        <axis xyz="1 0 0"/>
+        <origin rpy="0 0 0" xyz="0.042825 0 0"/>
         <parent link="$(arg robot_name)/base_gripper_link"/>
         <child link="$(arg robot_name)/end_effector_link"/>
