Commit message: Change manipulator description to conform to DH parameters

File: manipulator_unal_description/urdf/manipulator_backup1.urdf.xacro (robot description, xacro)
@@ -126,5 +126,5 @@
         <axis xyz="0 0 1"/>
         <limit effort="100" lower="${radians(-92)}" upper="${radians(101)}" velocity="${pi}"/>
-        <origin rpy="${pi} 0 ${-pi/2}" xyz="0.05955 -0.3 0.0"/>
+        <origin rpy="${pi} 0 0" xyz="0.05955 -0.3 0.0"/>
         <parent link="$(arg robot_name)/upper_arm_link"/>
         <child link="$(arg robot_name)/upper_forearm_link"/>
@@ -133,5 +133,5 @@
     <link name="$(arg robot_name)/upper_forearm_link">
         <visual>
-            <origin rpy="${pi/2} 0 ${-pi/2}" xyz="0 0 0"/>
+            <origin rpy="${pi/2} 0 0" xyz="0 0 0"/>
             <geometry>
                 <mesh filename="package://manipulator_unal_description/meshes/VXSA-300-M-4-UF.stl" scale="0.001 0.001 0.001"/>
@@ -140,5 +140,5 @@
         </visual>
         <collision>
-            <origin rpy="${pi/2} 0 ${-pi/2}" xyz="0 0 0"/>
+            <origin rpy="${pi/2} 0 0" xyz="0 0 0"/>
             <geometry>
                 <mesh filename="package://manipulator_unal_description/meshes/VXSA-300-M-4-UF.stl" scale="0.001 0.001 0.001"/>
@@ -146,5 +146,5 @@
         </collision>
         <inertial>
-            <origin rpy="${pi/2} 0 ${-pi/2}" xyz="0 -0.105723 0"/>
+            <origin rpy="${pi/2} 0 0" xyz="0.105723 0 0"/>
             <mass value="0.322228" />
             <inertia    ixx="0.0001524000"
@@ -160,5 +160,5 @@
         <axis xyz="0 0 1"/>
         <limit effort="100" lower="${radians(-180)}" upper="${radians(180)}" velocity="${pi}"/>
-        <origin rpy="${pi/2} 0 0" xyz="0 -0.2 0"/>
+        <origin rpy="${pi/2} 0 ${pi/2}" xyz="0.2 0 0"/>
         <parent link="$(arg robot_name)/upper_forearm_link"/>
         <child link="$(arg robot_name)/lower_forearm_link"/>
@@ -194,5 +194,5 @@
         <axis xyz="0 0 1"/>
         <limit effort="100" lower="${radians(-130)}" upper="${radians(107)}" velocity="${pi}"/>
-        <origin rpy="${-pi/2} 0 0" xyz="0 0 0.1"/>
+        <origin rpy="${-pi/2} ${-pi/2} 0" xyz="0 0 0.1"/>
         <parent link="$(arg robot_name)/lower_forearm_link"/>
         <child link="$(arg robot_name)/wrist_link"/>
@@ -201,5 +201,5 @@
     <link name="$(arg robot_name)/wrist_link">
         <visual>
-            <origin rpy="0 ${pi/2} 0" xyz="0 0 0"/>
+            <origin rpy="0 ${pi/2} ${pi/2}" xyz="0 0 0"/>
             <geometry>
                 <mesh filename="package://manipulator_unal_description/meshes/VXSA-300-M-6-Wrist.stl" scale="0.001 0.001 0.001"/>
@@ -208,5 +208,5 @@
         </visual>
         <collision>
-            <origin rpy="0 ${pi/2} 0" xyz="0 0 0"/>
+            <origin rpy="0 ${pi} ${pi/2}" xyz="0 0 0"/>
             <geometry>
                 <mesh filename="package://manipulator_unal_description/meshes/VXSA-300-M-6-Wrist.stl" scale="0.001 0.001 0.001"/>
@@ -214,5 +214,5 @@
         </collision>
         <inertial>
-            <origin rpy="0 ${pi/2} 0" xyz="0.0105650000 -0.0467430000 0.0000076652"/>
+            <origin rpy="0 ${pi} ${pi/2}" xyz="0.0467430000 0.0105650000 0.0000076652"/>
             <mass value="0.115395" />
             <inertia    ixx="0.0000463100"
@@ -228,5 +228,5 @@
         <axis xyz="0 0 1"/>
         <limit effort="100" lower="${-pi}" upper="${pi}" velocity="${pi}"/>
-        <origin rpy="${pi/2} ${pi} 0" xyz="0 -0.069744 0"/>
+        <origin rpy="${-pi/2} 0 ${-pi/2}" xyz="0.069744 0 0"/>
         <parent link="$(arg robot_name)/wrist_link"/>
         <child link="$(arg robot_name)/base_gripper_link"/>

File: mobile_manipulator_unal_description/urdf/mobile_manipulator.urdf (robot description, URDF)
Before this commit: robot mobile_robot, 21 links, 20 joints
Joints:
- joint elbow_joint: origin xyz=0.05955 -0.3 0.0 rpy=3.14159265359 0 0 -> xyz=0.05955 -0.3 0.0 rpy=3.14159265359 0 -1.57079632679
- joint lower_forearm_joint: origin xyz=0 0 0.1 rpy=-1.57079632679 -1.57079632679 0 -> xyz=0 0 0.1 rpy=-1.57079632679 0 0
- joint upper_forearm_joint: origin xyz=0.2 0 0 rpy=1.57079632679 0 1.57079632679 -> xyz=0 -0.2 0 rpy=1.57079632679 0 0
- joint wrist_joint: origin xyz=0.069744 0 0 rpy=-1.57079632679 0 -1.57079632679 -> xyz=0 -0.069744 0 rpy=1.57079632679 3.14159265359 0
