Commit message: Fixed limits in joints for manipulator

File: manipulator_unal_description/urdf/manipulator.urdf.xacro (robot description, xacro)
@@ -57,5 +57,5 @@
     <joint name="waist_joint" type="revolute">
         <axis xyz="0 0 1"/>
-        <limit effort="100" lower="${-pi}" upper="${pi}" velocity="${pi}"/>
+        <limit  lower="${-pi}" upper="${pi}" velocity="3.1" effort="10.6"/>
         <origin rpy="0 0 0" xyz="0 0 0.0787"/>
         <parent link="$(arg robot_name)/base_link"/>
@@ -91,5 +91,5 @@
     <joint name="shoulder_joint" type="revolute">
         <axis xyz="0 0 1"/>
-        <limit effort="100" lower="${radians(-106)}" upper="${radians(101)}" velocity="${pi}"/>
+        <limit lower="${radians(-106)}" upper="${radians(101)}" velocity="3.1" effort="21.2"/>
         <origin rpy="${-pi/2} 0 0" xyz="0 0 0.04805"/>
         <parent link="$(arg robot_name)/shoulder_link"/>
@@ -125,5 +125,5 @@
     <joint name="elbow_joint" type="revolute">
         <axis xyz="0 0 1"/>
-        <limit effort="100" lower="${radians(-92)}" upper="${radians(101)}" velocity="${pi}"/>
+        <limit lower="${radians(-92)}" upper="${radians(101)}" velocity="3.1" effort="21.2" />
         <origin rpy="${pi} 0 ${-pi/2}" xyz="0.05955 -0.3 0.0"/>
         <parent link="$(arg robot_name)/upper_arm_link"/>
@@ -159,5 +159,5 @@
     <joint name="upper_forearm_joint" type="revolute">
         <axis xyz="0 0 1"/>
-        <limit effort="100" lower="${radians(-180)}" upper="${radians(180)}" velocity="${pi}"/>
+        <limit lower="${radians(-180)}" upper="${radians(180)}" velocity="3.1" effort="10.6"/>
         <origin rpy="${pi/2} 0 0" xyz="0 -0.2 0"/>
         <parent link="$(arg robot_name)/upper_forearm_link"/>
@@ -193,5 +193,5 @@
     <joint name="lower_forearm_joint" type="revolute">
         <axis xyz="0 0 1"/>
-        <limit effort="100" lower="${radians(-130)}" upper="${radians(107)}" velocity="${pi}"/>
+        <limit lower="${radians(-130)}" upper="${radians(107)}" velocity="3.1" effort="10.6" />
         <origin rpy="${-pi/2} 0 0" xyz="0 0 0.1"/>
         <parent link="$(arg robot_name)/lower_forearm_link"/>
@@ -227,5 +227,5 @@
     <joint name="wrist_joint" type="revolute">
         <axis xyz="0 0 1"/>
-        <limit effort="100" lower="${-pi}" upper="${pi}" velocity="${pi}"/>
+        <limit lower="${-pi}" upper="${pi}" velocity="3.1" effort="4.1"/>
         <origin rpy="${pi/2} ${pi} 0" xyz="0 -0.069744 0"/>
         <parent link="$(arg robot_name)/wrist_link"/>
