Commit message: Added a parsing of the XACRO file at the beginnig of the mobile manipulator Gazebo file

File: mobile_manipulator_unal_description/urdf/mobile_manipulator.urdf (robot description, URDF)
Before this commit: robot mobile_robot, 20 links, 19 joints
Links:
- added link mobile_manipulator/imu_link
Joints:
- added joint imu_joint: type fixed, parent mobile_manipulator/mobile_base_link, child mobile_manipulator/imu_link, origin xyz=0.0 -0.06 0.10 rpy=0 0 0
- joint elbow_joint: axis 0 1 0 -> 0 0 1; origin xyz=0.05955 0 0.3 rpy=3.14159265359 0 0 -> xyz=0.05955 -0.3 0.0 rpy=3.14159265359 0 0
- joint lower_forearm_joint: axis 0 1 0 -> 0 0 1; origin xyz=0.1 0 0 rpy=0 0 0 -> xyz=0 0 0.1 rpy=-1.57079632679 -1.57079632679 0
- joint shoulder_joint: axis 0 1 0 -> 0 0 1; origin xyz=0 0 0.04805 rpy=0 0 0 -> xyz=0 0 0.04805 rpy=-1.57079632679 0 0
- joint tcp_joint: axis 1 0 0 -> (none); origin xyz=0.042825 0 0 rpy=0 0 0 -> xyz=0.0 0 0.042825 rpy=0 -1.57079632679 0
- joint upper_forearm_joint: axis 1 0 0 -> 0 0 1; origin xyz=0.2 0 0 rpy=0 0 0 -> xyz=0.2 0 0 rpy=1.57079632679 0 1.57079632679
- joint wrist_joint: axis 1 0 0 -> 0 0 1; origin xyz=0.069744 0 0 rpy=-3.14159265359 0 0 -> xyz=0.069744 0 0 rpy=-1.57079632679 0 -1.57079632679

Commit message: Checked OSC with new effort limits

File: mobile_manipulator_unal_description/urdf/mobile_manipulator.urdf (robot description, URDF)
Before this commit: robot mobile_robot, 21 links, 20 joints
Joints:
- joint elbow_joint: limit lower=-1.60570291183 upper=1.76278254451 effort=100 velocity=3.14159265359 -> lower=-1.60570291183 upper=1.76278254451 effort=21.2 velocity=3.1
- joint lower_forearm_joint: limit lower=-2.26892802759 upper=1.86750229963 effort=100 velocity=3.14159265359 -> lower=-2.26892802759 upper=1.86750229963 effort=10.6 velocity=3.1
- joint shoulder_joint: limit lower=-1.85004900711 upper=1.76278254451 effort=100 velocity=3.14159265359 -> lower=-1.85004900711 upper=1.76278254451 effort=21.2 velocity=3.1
- joint upper_forearm_joint: limit lower=-3.14159265359 upper=3.14159265359 effort=100 velocity=3.14159265359 -> lower=-3.14159265359 upper=3.14159265359 effort=10.6 velocity=3.1
- joint waist_joint: limit lower=-3.14159265359 upper=3.14159265359 effort=100 velocity=3.14159265359 -> lower=-3.14159265359 upper=3.14159265359 effort=10.6 velocity=3.1
- joint wrist_joint: limit lower=-3.14159265359 upper=3.14159265359 effort=100 velocity=3.14159265359 -> lower=-3.14159265359 upper=3.14159265359 effort=4.1 velocity=3.1

Commit message: Testing noetic

File: mobile_manipulator_unal_description/urdf/mobile_manipulator.urdf (robot description, URDF)
Before this commit: robot mobile_robot, 21 links, 20 joints
Joints:
- joint elbow_joint: limit lower=-1.60570291183 upper=1.76278254451 effort=21.2 velocity=3.1 -> lower=-1.6057029118347832 upper=1.7627825445142729 effort=21.2 velocity=3.1; origin xyz=0.05955 -0.3 0.0 rpy=3.14159265359 0 -1.57079632679 -> xyz=0.05955 -0.3 0.0 rpy=3.141592653589793 0 -1.5707963267948966
- joint gripper_joint: limit effort=100 velocity=3.14159265359 -> effort=100 velocity=3.141592653589793
- joint lower_forearm_joint: limit lower=-2.26892802759 upper=1.86750229963 effort=10.6 velocity=3.1 -> lower=-2.2689280275926285 upper=1.8675022996339325 effort=10.6 velocity=3.1; origin xyz=0 0 0.1 rpy=-1.57079632679 0 0 -> xyz=0 0 0.1 rpy=-1.5707963267948966 0 0
- joint shoulder_joint: limit lower=-1.85004900711 upper=1.76278254451 effort=21.2 velocity=3.1 -> lower=-1.8500490071139892 upper=1.7627825445142729 effort=21.2 velocity=3.1; origin xyz=0 0 0.04805 rpy=-1.57079632679 0 0 -> xyz=0 0 0.04805 rpy=-1.5707963267948966 0 0
- joint tcp_joint: origin xyz=0.0 0 0.042825 rpy=0 -1.57079632679 0 -> xyz=0.0 0 0.042825 rpy=0 -1.5707963267948966 0
- joint upper_forearm_joint: limit lower=-3.14159265359 upper=3.14159265359 effort=10.6 velocity=3.1 -> lower=-3.141592653589793 upper=3.141592653589793 effort=10.6 velocity=3.1; origin xyz=0 -0.2 0 rpy=1.57079632679 0 0 -> xyz=0 -0.2 0 rpy=1.5707963267948966 0 0
- joint waist_joint: limit lower=-3.14159265359 upper=3.14159265359 effort=10.6 velocity=3.1 -> lower=-3.141592653589793 upper=3.141592653589793 effort=10.6 velocity=3.1
- joint wrist_joint: limit lower=-3.14159265359 upper=3.14159265359 effort=4.1 velocity=3.1 -> lower=-3.141592653589793 upper=3.141592653589793 effort=4.1 velocity=3.1; origin xyz=0 -0.069744 0 rpy=1.57079632679 3.14159265359 0 -> xyz=0 -0.069744 0 rpy=1.5707963267948966 3.141592653589793 0
